Commit message: Uptade 20 March

File: src/my_robotino_urdf/urdf/robotino_body.xacro (robot description, xacro)
@@ -49,10 +49,10 @@
       <origin xyz="0.008 0 0.137" rpy="0 0 ${M_PI/2}"/>
     </anglebracketusb>
+    <!--laser name="laser" parent="base_link">
+      <origin xyz="-0.022 0 0.232" rpy="0 0 0"/>
+    </laser-->
     <laser name="laser" parent="base_link">
-      <origin xyz="-0.022 0 0.232" rpy="0 0 0"/>
+      <origin xyz="0.155 0 ${BASE_HEIGHT/2}" rpy="0 0 0"/>
     </laser>
-    <!--laser name="laser" parent="base_link"-->
-      <!--origin xyz="0.12 0 ${BASE_HEIGHT/2}" rpy="0 0 0"/-->
-    <!--/laser-->
   </macro>
 </robot>

File: src/my_robotino_urdf/urdf/robotino_hardware.xacro (robot description, xacro)
@@ -3,6 +3,6 @@
   <property name="M_PI" value="3.14159"/>
   <property name="M_SCALE" value="0.01"/>
-  <property name="HOKUYO_RADIUS" value="0.02"/>
-  <property name="HOKUYO_LENGTH" value="0.07"/>
+  <property name="HOKUYO_RADIUS" value="0.0002"/>
+  <property name="HOKUYO_LENGTH" value="0.0007"/>
   <property name="KINECT_LENGTH" value="0.064"/>
   <property name="KINECT_WIDTH" value="0.121"/>
@@ -73,5 +73,5 @@
         <origin xyz="0 0 0" rpy="0 0 ${M_PI/2}" />
         <geometry>
-          <mesh filename="package://my_robotino_urdf/meshes/RobotinoLaserScanner.dae" scale="${M_SCALE} ${M_SCALE} ${M_SCALE}"/>
+          <mesh filename="package://my_robotino_urdf/meshes/RobotinoLaserScanner.dae" scale="0.001 0.001 0.001"/>
         </geometry>
       </visual>

Commit message: Adding controller, 22 March

File: src/my_robotino_urdf/urdf/robotino_body.xacro (robot description, xacro)
@@ -55,4 +55,28 @@
       <origin xyz="0.155 0 ${BASE_HEIGHT/2}" rpy="0 0 0"/>
     </laser>
+    <laser name="laser1" parent="base_link">
+      <origin xyz="0.11873 0.09963 ${BASE_HEIGHT/2}" rpy="0 0 ${M_PI/4.5}"/>
+    </laser>
+    <laser name="laser2" parent="base_link">
+      <origin xyz="0.11873 -0.099630 ${BASE_HEIGHT/2}" rpy="0 0 -${M_PI/4.5}"/>
+    </laser>
+    <laser name="laser3" parent="base_link">
+      <origin xyz="0.02691 0.15264 ${BASE_HEIGHT/2}" rpy="0 0 ${M_PI/2.25}"/>
+    </laser>
+    <laser name="laser4" parent="base_link">
+      <origin xyz="0.02691 -0.15264 ${BASE_HEIGHT/2}" rpy="0 0 -${M_PI/2.25}"/>
+    </laser>
+    <laser name="laser5" parent="base_link">
+      <origin xyz="-0.0775 0.13423 ${BASE_HEIGHT/2}" rpy="0 0 ${M_PI/1.5}"/>
+    </laser>
+    <laser name="laser6" parent="base_link">
+      <origin xyz="-0.0775 -0.13423 ${BASE_HEIGHT/2}" rpy="0 0 -${M_PI/1.5}"/>
+    </laser>
+    <laser name="laser7" parent="base_link">
+      <origin xyz="-0.14565 0.05301 ${BASE_HEIGHT/2}" rpy="0 0 ${M_PI/1.125}"/>
+    </laser>
+    <laser name="laser8" parent="base_link">
+      <origin xyz="-0.14565 -0.05301 ${BASE_HEIGHT/2}" rpy="0 0 -${M_PI/1.125}"/>
+    </laser>
   </macro>
 </robot>

File: src/my_robotino_urdf/urdf/robotino_hardware.xacro (robot description, xacro)
@@ -57,10 +57,10 @@
   <!-- LASER SCANNER -->
   <macro name="laser" params="parent name *origin">
-    <joint name="hokuyo_joint" type="fixed">
+    <joint name="${name}_joint" type="fixed">
       <insert_block name="origin" />
       <parent link="${parent}"/>
-      <child link="hokuyo_link" />
+      <child link="${name}_link" />
     </joint>
-    <link name="hokuyo_link">
+    <link name="${name}_link">
       <inertial>
         <mass value="0.00001" />
